File: Driver velocidad DCmotor.brd (EAGLE design)
At the start: 47.7 x 55.4 mm, 11 parts

Commit message: se agrega la resistencia de 330 Ohms a la compuerta del MOSFET
Parts:
- added R5: 330, adafruit:M1206
Connections:
- new net N$15: R5.1, U$1.D3
- net N$8: now also R5.2; no longer U$1.D3
Routing:
- net N$8: track 35.9 -> 0.00 mm
- net N$15: track 0.00 -> 28.8 mm
- net N$14: track 0.00 -> 4.57 mm
Changed lines of the file:
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@@
 <element name="T2" library="transistor" package="SOT23-BEC" value="" x="59.944" y="15.24"/>
 <element name="U$1" library="adafruit" package="ARDUINO-NOHOLE" value="ARDUINO-NOHOLE" x="12.7" y="2.54"/>
+<element name="R5" library="adafruit" package="M1206" value="330" x="65.278" y="24.638" rot="R270"/>
 </elements>
 <signals>
@@
 </signal>
 <signal name="N$8">
-<wire x1="65.278" y1="18.796" x2="65.278" y2="46.228" width="1.016" layer="1"/>
-<wire x1="65.278" y1="46.228" x2="68.58" y2="49.53" width="1.016" layer="1"/>
 <contactref element="T1" pad="1"/>
-<contactref element="U$1" pad="D3"/>
-<wire x1="68.58" y1="49.53" x2="68.58" y2="53.34" width="1.016" layer="1"/>
-<wire x1="65.4812" y1="18.8214" x2="65.278" y2="18.796" width="0" layer="19" extent="1-1"/>
+<contactref element="R5" pad="2"/>
+<wire x1="65.278" y1="23.238" x2="65.4812" y2="18.8214" width="0" layer="19" extent="1-1"/>
 </signal>
 <signal name="N$3">
@@
 <wire x1="58.166" y1="27.054" x2="58.166" y2="26.924" width="0" layer="19" extent="1-1"/>
 </signal>
+<signal name="N$14">
+<wire x1="65.024" y1="18.542" x2="65.024" y2="23.114" width="1.016" layer="1"/>
+</signal>
+<signal name="N$15">
+<wire x1="65.278" y1="25.908" x2="65.278" y2="46.736" width="1.016" layer="1"/>
+<wire x1="65.278" y1="46.736" x2="68.58" y2="50.038" width="1.016" layer="1"/>
+<contactref element="U$1" pad="D3"/>
+<contactref element="R5" pad="1"/>
+<wire x1="65.278" y1="26.038" x2="68.58" y2="53.34" width="0" layer="19" extent="1-1"/>
+<wire x1="68.58" y1="50.038" x2="68.58" y2="53.34" width="1.016" layer="1"/>
+</signal>
 </signals>
